Commit message: Fixed a discrepancy between the prediction and simulation model by adding quadcopter mass into thrust command calculation

File: config/hummingbird.xacro (robot description, xacro)
@@ -31,5 +31,8 @@
   <xacro:property name="radius_rotor" value="0.1" /> <!-- [m] -->
   <xacro:property name="motor_constant" value="8.54858e-06" /> <!-- [kg m/s^2] -->
-  <xacro:property name="moment_constant" value="0.05" /> <!-- [m] 0.016-->
+  <!--
+  <xacro:property name="moment_constant" value="0.05" />
+  -->
+  <xacro:property name="moment_constant" value="0.016" /> <!-- [m] 0.016-->
   <xacro:property name="time_constant_up" value="0.0125" /> <!-- [s] -->
   <xacro:property name="time_constant_down" value="0.025" /> <!-- [s] -->
